File: Hardware/PCB/Final_V1/Final_PCB/attiny.kicad_sch (KiCad schematic)
At the start: 6 parts, among them IC3 ATTINY85-20SFR, J2 Conn_ARM_SWD_TagConnect_TC203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

Commit message: fixed Schematics
Connections:
- net PIN_5: now also S1.1 (NO)
- net VCC: no longer S1.1 (NO)
Other:
- moved on the sheet: R10, R9, S1, S2
Changed lines of the file:
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@@
 	(text "Switches"
 		(exclude_from_sim no)
-		(at 205.232 90.17 0)
+		(at 215.392 33.02 0)
 		(effects
 			(font
@@
 	)
 	(junction
-		(at 227.33 64.77)
+		(at 229.87 44.45)
 		(diameter 0)
 		(color 0 0 0 0)
@@
 	)
 	(junction
-		(at 190.5 64.77)
+		(at 237.49 24.13)
 		(diameter 0)
 		(color 0 0 0 0)
 	)
-	(junction
-		(at 227.33 81.28)
-		(diameter 0)
-		(color 0 0 0 0)
-	)
 	(no_connect
 		(at 64.77 67.31)
@@
 	(wire
 		(pts
-			(xy 187.96 81.28) (xy 194.31 81.28)
-		)
-		(stroke
-			(width 0)
-			(type default)
-		)
-	)
-	(wire
-		(pts
-			(xy 227.33 81.28) (xy 234.95 81.28)
+			(xy 198.12 24.13) (xy 204.47 24.13)
+		)
+		(stroke
+			(width 0)
+			(type default)
+		)
+	)
+	(wire
+		(pts
+			(xy 237.49 24.13) (xy 245.11 24.13)
 		)
 		(stroke
@@
 	(wire
 		(pts
-			(xy 227.33 64.77) (xy 234.95 64.77)
+			(xy 229.87 44.45) (xy 237.49 44.45)
 		)
 		(stroke
@@
 	(wire
 		(pts
-			(xy 227.33 53.34) (xy 227.33 57.15)
+			(xy 199.39 44.45) (xy 204.47 44.45)
+		)
+		(stroke
+			(width 0)
+			(type default)
+		)
+	)
+	(wire
+		(pts
+			(xy 229.87 33.02) (xy 229.87 36.83)
 		)
 		(stroke
@@
 	(wire
 		(pts
-			(xy 190.5 64.77) (xy 195.58 64.77)
-		)
-		(stroke
-			(width 0)
-			(type default)
-		)
-	)
-	(wire
-		(pts
 			(xy 168.91 41.91) (xy 175.26 41.91)
 		)
@@
 	(wire
 		(pts
-			(xy 220.98 64.77) (xy 227.33 64.77)
-		)
-		(stroke
-			(width 0)
-			(type default)
-		)
-	)
-	(wire
-		(pts
 			(xy 57.15 72.39) (xy 57.15 76.2)
 		)
@@
 	(wire
 		(pts
-			(xy 227.33 69.85) (xy 227.33 73.66)
-		)
-		(stroke
-			(width 0)
-			(type default)
-		)
-	)
-	(wire
-		(pts
-			(xy 219.71 81.28) (xy 227.33 81.28)
+			(xy 237.49 13.97) (xy 237.49 16.51)
+		)
+		(stroke
+			(width 0)
+			(type default)
+		)
+	)
+	(wire
+		(pts
+			(xy 229.87 24.13) (xy 237.49 24.13)
 		)
 		(stroke
@@
 	)
 	(label "PIN_7"
-		(at 187.96 81.28 0)
+		(at 198.12 24.13 0)
 		(effects
 			(font
@@
 	(label "PIN_1"
 		(at 49.53 64.77 0)
+		(effects
+			(font
+				(size 1.27 1.27)
+			)
+			(justify left bottom)
+		)
+	)
+	(label "PIN_5"
+		(at 199.39 44.45 0)
 		(effects
 			(font
@@
 	(hierarchical_label "VCC"
 		(shape input)
-		(at 227.33 53.34 0)
+		(at 229.87 33.02 0)
 		(effects
 			(font
@@
 	(hierarchical_label "SDA"
 		(shape input)
-		(at 234.95 81.28 0)
+		(at 245.11 24.13 0)
 		(effects
 			(font
@@
 	(hierarchical_label "VCC"
 		(shape input)
-		(at 227.33 69.85 0)
+		(at 237.49 13.97 0)
 		(effects
 			(font
@@
 	(hierarchical_label "SCL"
 		(shape input)
-		(at 234.95 64.77 0)
+		(at 237.49 44.45 0)
 		(effects
 			(font
@@
 	(symbol
 		(lib_id "Device:R")
-		(at 227.33 60.96 0)
+		(at 229.87 40.64 0)
 		(unit 1)
 		(exclude_from_sim no)
@@
 		(fields_autoplaced yes)
 		(property "Reference" "R9"
-			(at 229.87 59.6899 0)
+			(at 232.41 39.3699 0)
 			(effects
 				(font
@@
 		)
 		(property "Value" "10k"
-			(at 229.87 62.2299 0)
+			(at 232.41 41.9099 0)
 			(effects
 				(font
@@
 		)
 		(property "Footprint" ""
-			(at 225.552 60.96 90)
+			(at 228.092 40.64 90)
 			(effects
 				(font
@@
 		)
 		(property "Datasheet" "~"
-			(at 227.33 60.96 0)
+			(at 229.87 40.64 0)
 			(effects
 				(font
@@
 		)
 		(property "Description" "Resistor"
-			(at 227.33 60.96 0)
+			(at 229.87 40.64 0)
 			(effects
 				(font
@@
 	(symbol
 		(lib_id "Device:R")
-		(at 227.33 77.47 0)
+		(at 237.49 20.32 0)
 		(unit 1)
 		(exclude_from_sim no)
@@
 		(on_board yes)
 		(dnp no)
-		(fields_autoplaced yes)
 		(property "Reference" "R10"
-			(at 229.87 76.1999 0)
+			(at 240.03 19.0499 0)
 			(effects
 				(font
@@
 		)
 		(property "Value" "10k"
-			(at 229.87 78.7399 0)
+			(at 240.03 21.5899 0)
 			(effects
 				(font
@@
 		)
 		(property "Footprint" ""
-			(at 225.552 77.47 90)
+			(at 235.712 20.32 90)
 			(effects
 				(font
@@
 		)
 		(property "Datasheet" "~"
-			(at 227.33 77.47 0)
+			(at 237.49 20.32 0)
 			(effects
 				(font
@@
 		)
 		(property "Description" "Resistor"
-			(at 227.33 77.47 0)
+			(at 237.49 20.32 0)
 			(effects
 				(font
@@
 	(symbol
 		(lib_id "CAS-120A1:CAS-120A1")
-		(at 194.31 81.28 0)
+		(at 204.47 24.13 0)
 		(unit 1)
 		(exclude_from_sim no)
@@
 		(fields_autoplaced yes)
 		(property "Reference" "S2"
-			(at 207.01 73.66 0)
+			(at 217.17 16.51 0)
 			(effects
 				(font
@@
 		)
 		(property "Value" "CAS-120A1"
-			(at 207.01 76.2 0)
+			(at 217.17 19.05 0)
 			(effects
 				(font
@@
 		)
 		(property "Footprint" "CAS120A1"
-			(at 215.9 176.2 0)
+			(at 226.06 119.05 0)
 			(effects
 				(font
@@
 		)
 		(property "Datasheet" "https://www.nidec-copal-electronics.com/e/catalog/switch/cas.pdf"
-			(at 215.9 276.2 0)
+			(at 226.06 219.05 0)
 			(effects
 				(font
@@
 		)
 		(property "Description" "Surface Mount Slide Switch Single Pole Double Throw (SPDT) 100 (Non-Switching) mA, 100 (Switching) mA Slide"
-			(at 194.31 81.28 0)
+			(at 204.47 24.13 0)
 			(effects
 				(font
@@
 		)
 		(property "Height" "2.5"
-			(at 215.9 476.2 0)
+			(at 226.06 419.05 0)
 			(effects
 				(font
@@
 		)
 		(property "Mouser Part Number" "229-CAS-120A1"
-			(at 215.9 576.2 0)
+			(at 226.06 519.05 0)
 			(effects
 				(font
@@
 		)
 		(property "Mouser Price/Stock" "https://www.mouser.co.uk/ProductDetail/Nidec-Components/CAS-120A1?qs=XeJtXLiO41SLHVe%252BE1BF5w%3D%3D"
-			(at 215.9 676.2 0)
+			(at 226.06 619.05 0)
 			(effects
 				(font
@@
 		)
 		(property "Manufacturer_Name" "Nidec Copal"
-			(at 215.9 776.2 0)
+			(at 226.06 719.05 0)
 			(effects
 				(font
@@
 		)
 		(property "Manufacturer_Part_Number" "CAS-120A1"
-			(at 215.9 876.2 0)
+			(at 226.06 819.05 0)
 			(effects
 				(font
@@
 	(symbol
 		(lib_id "CAS-120A1:CAS-120A1")
-		(at 195.58 64.77 0)
+		(at 204.47 44.45 0)
 		(unit 1)
 		(exclude_from_sim no)
@@
 		(fields_autoplaced yes)
 		(property "Reference" "S1"
-			(at 208.28 57.15 0)
+			(at 217.17 36.83 0)
 			(effects
 				(font
@@
 		)
 		(property "Value" "CAS-120A1"
-			(at 208.28 59.69 0)
+			(at 217.17 39.37 0)
 			(effects
 				(font
@@
 		)
 		(property "Footprint" "CAS120A1"
-			(at 217.17 159.69 0)
+			(at 226.06 139.37 0)
 			(effects
 				(font
@@
 		)
 		(property "Datasheet" "https://www.nidec-copal-electronics.com/e/catalog/switch/cas.pdf"
-			(at 217.17 259.69 0)
+			(at 226.06 239.37 0)
 			(effects
 				(font
@@
 		)
 		(property "Description" "Surface Mount Slide Switch Single Pole Double Throw (SPDT) 100 (Non-Switching) mA, 100 (Switching) mA Slide"
-			(at 195.58 64.77 0)
+			(at 204.47 44.45 0)
 			(effects
 				(font
@@
 		)
 		(property "Height" "2.5"
-			(at 217.17 459.69 0)
+			(at 226.06 439.37 0)
 			(effects
 				(font
@@
 		)
 		(property "Mouser Part Number" "229-CAS-120A1"
-			(at 217.17 559.69 0)
+			(at 226.06 539.37 0)
 			(effects
 				(font
@@
 		)
 		(property "Mouser Price/Stock" "https://www.mouser.co.uk/ProductDetail/Nidec-Components/CAS-120A1?qs=XeJtXLiO41SLHVe%252BE1BF5w%3D%3D"
-			(at 217.17 659.69 0)
+			(at 226.06 639.37 0)
 			(effects
 				(font
@@
 		)
 		(property "Manufacturer_Name" "Nidec Copal"
-			(at 217.17 759.69 0)
+			(at 226.06 739.37 0)
 			(effects
 				(font
@@
 		)
 		(property "Manufacturer_Part_Number" "CAS-120A1"
-			(at 217.17 859.69 0)
-			(effects
-				(font
+			(at 226.06 839.37 0)
+			(effects
+				(font

Commit message: fixed last commit, because it was wrong
Connections:
- net VCC renamed +3.3V
Other:
- moved on the sheet: R10, R9, S1, S2

Commit message: fixing xhematics
Parts:
- R10, R9: footprint (none) -> Resistor_SMD:R_0603_1608Metric
Changed lines of the file:
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@@
 			)
 		)
-		(property "Footprint" ""
+		(property "Footprint" "Resistor_SMD:R_0603_1608Metric"
 			(at 231.902 66.04 90)
 			(effects
@@
 			)
 		)
-		(property "Footprint" ""
+		(property "Footprint" "Resistor_SMD:R_0603_1608Metric"
 			(at 239.522 45.72 90)
 			(effects

Commit message: #1: Add footprints to the components
Parts:
- IC3: footprint SOIC127P798X216-8N -> custom:SOIC127P798X216-8N
- S1, S2: footprint CAS120A1 -> custom:CAS120A1
Changed lines of the file:
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@@
 			)
 		)
-		(property "Footprint" "SOIC127P798X216-8N"
+		(property "Footprint" "custom:SOIC127P798X216-8N"
 			(at 180.34 159.69 0)
 			(effects
@@
 			)
 		)
-		(property "Footprint" "CAS120A1"
+		(property "Footprint" "custom:CAS120A1"
 			(at 229.87 144.45 0)
 			(effects
@@
 			)
 		)
-		(property "Footprint" "CAS120A1"
+		(property "Footprint" "custom:CAS120A1"
 			(at 229.87 164.77 0)
 			(effects
