File: Hardware/PCB/Final_V1/Final_PCB/BMS.kicad_sch (KiCad schematic)
At the start: 8 parts, among them Q1 Q_NMOS_Depletion_DSG, Q2 Q_NMOS_Depletion_DSG, U2 BQ298xy

Commit message: added footprints for BQ298010RUGR and BSC009NE2LS5IATMA1
Parts:
- U2: footprint Fooprints:QFN50P150X150X40-8N -> custom:X2QFN
Connections:
- net at U2.1 (NC): now also RBAT1.2
Changed lines of the file:
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@@
 			)
 		)
-		(property "Footprint" "Fooprints:QFN50P150X150X40-8N"
+		(property "Footprint" "custom:X2QFN"
 			(at 129.794 90.678 0)
 			(effects

Commit message: started layouting
Parts:
- Q1, Q2: footprint Fooprints:MOSFET_BSC093N04LSGATMA1 -> custom:MOSFET_BSC093N04LSGATMA1
- U2: footprint custom:X2QFN -> custom:QFN50P150X150X40-8N
Connections:
- net at U2.1 (NC): now also RBAT1.2
Changed lines of the file:
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@@
 			)
 		)
-		(property "Footprint" "custom:X2QFN"
+		(property "Footprint" "custom:QFN50P150X150X40-8N"
 			(at 129.794 90.678 0)
 			(effects
@@
 			)
 		)
-		(property "Footprint" "Fooprints:MOSFET_BSC093N04LSGATMA1"
+		(property "Footprint" "custom:MOSFET_BSC093N04LSGATMA1"
 			(at 140.97 99.06 0)
 			(effects
@@
 			)
 		)
-		(property "Footprint" "Fooprints:MOSFET_BSC093N04LSGATMA1"
+		(property "Footprint" "custom:MOSFET_BSC093N04LSGATMA1"
 			(at 157.48 99.06 0)
 			(effects

Commit message: reapplied fixes because of commiting problems
Connections:
- net at U2.1 (NC): now also RBAT1.2
Changed lines of the file:
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@@
 	(wire
 		(pts
-			(xy 165.1 133.35) (xy 152.4 133.35)
+			(xy 168.91 133.35) (xy 152.4 133.35)
 		)
 		(stroke
@@
 	(hierarchical_label "BATT-"
 		(shape input)
-		(at 165.1 133.35 0)
+		(at 168.91 133.35 0)
 		(effects
 			(font

Commit message: #4: Layout-Session-17-11-25
Parts:
- removed RSENS1: 322, Resistor_SMD:R_2512_6332Metric, symbol Device:R
Connections:
- net PACK- is gone; now on net BATT-: CVDD1.2, U2.3 (VSS)
- net at U2.1 (NC): now also RBAT1.2
Changed lines of the file:
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@@
-	(wire
-		(pts
-			(xy 116.84 133.35) (xy 115.57 133.35)
-		)
-		(stroke
-			(width 0)
-			(type default)
-		)
-	)
 	(wire
 		(pts
@@
 		(pts
 			(xy 116.84 121.92) (xy 116.84 133.35)
+		)
+		(stroke
+			(width 0)
+			(type default)
+		)
+	)
+	(wire
+		(pts
+			(xy 107.95 133.35) (xy 116.84 133.35)
 		)
 		(stroke
@@
 					(unit 1)
 				)
-			)
-		)
-	)
-	(symbol
-		(lib_id "Device:R")
-		(at 111.76 133.35 90)
-		(unit 1)
-		(exclude_from_sim no)
-		(in_bom yes)
-		(on_board yes)
-		(dnp no)
-		(property "Reference" "RSENS1"
-			(at 113.284 131.572 0)
-			(effects
-				(font
-					(size 1.27 1.27)
-				)
-				(justify left)
-			)
-		)
-		(property "Value" "322"
-			(at 115.824 131.572 0)
-			(effects
-				(font
-					(size 1.27 1.27)
-				)
-				(justify left)
-				(hide yes)
-			)
-		)
-		(property "Footprint" "Resistor_SMD:R_2512_6332Metric"
-			(at 111.76 135.128 90)
-			(effects
-				(font
-					(size 1.27 1.27)
-				)
-				(hide yes)
-			)
-		)
-		(property "Datasheet" "~"
-			(at 111.76 133.35 0)
-			(effects
-				(font
-					(size 1.27 1.27)
-				)
-				(hide yes)
-			)
-		)
-		(property "Description" "Resistor"
-			(at 111.76 133.35 0)
-			(effects
-				(font
-					(size 1.27 1.27)
-				)
-				(hide yes)
-			)
-		)
-		(pin "1"
-		)
-		(pin "2"
-		)
-		(instances
-			(project "Final_PCB"
-				(path "/3cedac76-cdf6-4427-9720-a412bd9af7e2/46e274db-b5db-4871-9e0a-2907fab034b3"
-					(reference "RSENS1")
-					(unit 1)
-				)
