File: Hardware/PCB/Final_V1/Final_PCB/Gyro.kicad_sch (KiCad schematic)
At the start: 7 parts, among them U11 MPU-6050

Commit message: #4: Layout-Session-17-11-25
Parts:
- U11: footprint (none) -> Sensor_Motion:InvenSense_QFN-24_4x4mm_P0.5mm
Connections:
- net V3.3 renamed +3.3V
