File: Hardware/PCB/Final_V1/Final_PCB/Final_PCB.kicad_pcb (KiCad board)
At the start: 2 copper layers, 19.2 x 94 mm, 88 parts, among them IC1 BQ25895MRTWT, IC2 PCA9955BTWJ, IC3 ATTINY85-20SFR, J1 USB_C_Receptacle_USB2.0_16P, J2 Conn_ARM_SWD_TagConnect_TC203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, Q1 Q_NMOS_Depletion_DSG, Q2 Q_NMOS_Depletion_DSG, U1 TPS63000-Q1, U11 MPU-6050, U2 BQ298xy

Commit message: a few pcb edits
Parts:
- removed C10: 1u, Capacitor_SMD:C_0603_1608Metric
- removed C5, C9: 22u, Capacitor_SMD:C_0603_1608Metric
- removed TH1: Thermistor_NTC, Resistor_SMD:R_0603_1608Metric
Routing:
- net /BQ25895M/TS: track 35.3 -> 23.2 mm
- net FSYNC: track 9.91 -> 0.00 mm
- net /BQ25895M/REGN: track 23.9 -> 20.6 mm
- net /BQ25895M/VBus: track 70.4 -> 71.5 mm, vias 3 -> 5
- net +3.3V: track 48.9 -> 48.2 mm
- net Net-(IC2-LED11): track 77.9 -> 78.5 mm

Commit message: add pcb fixes
Parts:
- moved C11 2.45 mm to (139.2, 75.9)
- moved CVDD1 2.41 mm to (145.4, 114.5)
- moved R13 2.40 mm to (138.4, 72.2)
- moved R14 2.40 mm to (138.4, 74.1)
- moved Ra1 0.44 mm to (148.6, 127.3)
Routing:
- net GND: track 160.7 -> 128.4 mm
- net +3.3V: track 48.2 -> 34.3 mm, vias 18 -> 16
- net /BQ25895M/D+: track 60.0 -> 46.4 mm
- net /BQ25895M/Bat_Voltage: track 40.1 -> 35.0 mm
- net Net-(U2-VDD): track 16.4 -> 14.5 mm
- net Net-(IC2-LED10): track 86.1 -> 84.5 mm
- net Net-(IC2-LED1): track 14.0 -> 12.5 mm
- net Net-(IC2-LED2): track 16.0 -> 14.6 mm
- net Net-(Q2-G): track 12.5 -> 11.5 mm
- net Net-(IC2-LED11): track 78.5 -> 77.5 mm
- net Net-(J1-CC1): track 8.81 -> 8.14 mm
- net Net-(U1-EN): track 5.56 -> 6.21 mm
- net Net-(IC2-LED0): track 19.7 -> 20.3 mm
- net Net-(IC2-LED6): track 50.9 -> 50.4 mm
- net Net-(IC2-LED7): track 63.6 -> 64.1 mm, vias 3 -> 5
Other:
- board text added: "67"
- board text removed: "1"
- board text removed: "2"
